File: omega-dock-new.kicad_pcb (KiCad board)
At the start: 2 copper layers, 42.9 x 26.4 mm, 21 parts, among them J1 USB_A, J2 USB_PWR, J3 RJ45-TRAFO, U1 USBLC6-2, U2 AP111733, U3 OMEGA_2

Commit message: Update omega-dock-new.kicad_pcb
Other:
- board text added: "github.com/valerionew"
- board text removed: "github.com/5N44P"
Changed lines of the file:
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@@
   (gr_line (start 181.6608 47.752) (end 173.228 47.752) (layer F.SilkS) (width 0.1))
   (gr_line (start 181.6608 52.4764) (end 181.6608 47.752) (layer F.SilkS) (width 0.1))
-  (gr_text github.com/5N44P (at 188.0108 47.8536) (layer F.SilkS)
+  (gr_text github.com/valerionew (at 188.0108 47.8536) (layer F.SilkS)
     (effects (font (size 0.8 0.8) (thickness 0.15)))
   )
